Commit message: Changed urdf model to center the gripper. Figured out correct transformations for PyBullet world.

File: hsrb_description/robots/hand.urdf (robot description, URDF)
Before this commit: robot hsrb, 10 links, 9 joints
Joints:
- joint hand_palm_joint: origin xyz=0.012 0.0 0.1405 rpy=0.0 0.0 3.14159265359 -> xyz=0.012 0.0 0.0 rpy=0.0 0.0 3.14159265359
